Commit message: Updates and Bug Fixes as of 1/27/2020 - refer to the interbotix_ros_arms repo for details

File: interbotix_descriptions/urdf/vx300.urdf.xacro (robot description, xacro)
@@ -79,5 +79,5 @@
   <joint name="shoulder" type="revolute">
     <axis xyz="0 1 0"/>
-    <limit effort="100" lower="${radians(-101)}" upper="${radians(101)}" velocity="${pi}"/>
+    <limit effort="100" lower="${radians(-106)}" upper="${radians(101)}" velocity="${pi}"/>
     <origin rpy="0 0 0" xyz="0 0 0.04805"/>
     <parent link="$(arg robot_name)/shoulder_link"/>

File: interbotix_descriptions/urdf/vx300s.urdf.xacro (robot description, xacro)
@@ -79,5 +79,5 @@
   <joint name="shoulder" type="revolute">
     <axis xyz="0 1 0"/>
-    <limit effort="100" lower="${radians(-101)}" upper="${radians(101)}" velocity="${pi}"/>
+    <limit effort="100" lower="${radians(-106)}" upper="${radians(101)}" velocity="${pi}"/>
     <origin rpy="0 0 0" xyz="0 0 0.04805"/>
     <parent link="$(arg robot_name)/shoulder_link"/>
@@ -131,5 +131,5 @@
   <link name="$(arg robot_name)/upper_forearm_link">
     <visual>
-      <origin rpy="${pi/2} 0 ${pi/2}" xyz="0.165677 -0.037 0"/>
+      <origin rpy="0 0 0" xyz="0 0 0"/>
       <geometry>
         <mesh filename="package://interbotix_descriptions/meshes/meshes_vx300s/VXSA-300-M-4-UF.stl" scale="0.001 0.001 0.001"/>
@@ -138,5 +138,5 @@
     </visual>
     <collision>
-      <origin rpy="${pi/2} 0 ${pi/2}" xyz="0.165677 -0.037 0"/>
+      <origin rpy="0 0 0" xyz="0 0 0"/>
       <geometry>
         <mesh filename="package://interbotix_descriptions/meshes/meshes_vx300s/VXSA-300-M-4-UF.stl" scale="0.001 0.001 0.001"/>
@@ -144,7 +144,7 @@
     </collision>
     <inertial>
-      <origin rpy="${pi/2} 0 ${pi/2}" xyz="0 0 0"/>
-      <mass value="0.1" />
-      <inertia ixx="0.005" iyy="0.0002" izz="0.005" ixy="0" ixz="0" iyz="0" />
+      <origin rpy="0 0 0" xyz="0.105723 0 0"/>
+      <mass value="0.322228" />
+      <inertia ixx="0.0001524000" iyy="0.0013420000" izz="0.0014410000" ixy="-0.0000188300" ixz="-0.0000084064" iyz="0.0000012564" />
     </inertial>
   </link>
@@ -152,5 +152,5 @@
     <axis xyz="1 0 0"/>
     <limit effort="100" lower="${radians(-180)}" upper="${radians(180)}" velocity="${pi}"/>
-    <origin rpy="0 0 0" xyz="0.204929 0 0"/>
+    <origin rpy="0 0 0" xyz="0.2 0 0"/>
     <parent link="$(arg robot_name)/upper_forearm_link"/>
     <child link="$(arg robot_name)/lower_forearm_link"/>
@@ -167,5 +167,5 @@
   <link name="$(arg robot_name)/lower_forearm_link">
     <visual>
-      <origin rpy="${pi/2} ${pi/2} ${pi/2}" xyz="-0.039252 0 0.0365"/>
+      <origin rpy="0 0 0" xyz="0 0 0"/>
       <geometry>
         <mesh filename="package://interbotix_descriptions/meshes/meshes_vx300s/VXSA-300-M-5-LF.stl" scale="0.001 0.001 0.001"/>
@@ -174,5 +174,5 @@
     </visual>
     <collision>
-      <origin rpy="${pi/2} ${pi/2} ${pi/2}" xyz="-0.039252 0 0.0365"/>
+      <origin rpy="0 0 0" xyz="0 0 0"/>
       <geometry>
         <mesh filename="package://interbotix_descriptions/meshes/meshes_vx300s/VXSA-300-M-5-LF.stl" scale="0.001 0.001 0.001"/>
@@ -180,7 +180,7 @@
     </collision>
     <inertial>
-      <origin rpy="${pi/2} ${pi/2} ${pi/2}" xyz="0 0 0"/>
-      <mass value="0.1" />
-      <inertia ixx="0.005" iyy="0.0002" izz="0.005" ixy="0" ixz="0" iyz="0" />
+      <origin rpy="0 0 0" xyz="0.0513477000 -0.0068046200 0"/>
+      <mass value="0.414823" />
+      <inertia ixx="0.0001753000" iyy="0.0005269000" izz="0.0005911000" ixy="-0.0000852800" ixz="0" iyz="0" />
     </inertial>
   </link>
@@ -188,5 +188,5 @@
     <axis xyz="0 1 0"/>
     <limit effort="100" lower="${radians(-130)}" upper="${radians(107)}" velocity="${pi}"/>
-    <origin rpy="0 0 0" xyz="0.09545 0 0"/>
+    <origin rpy="0 0 0" xyz="0.1 0 0"/>
     <parent link="$(arg robot_name)/lower_forearm_link"/>
     <child link="$(arg robot_name)/wrist_link"/>

File: interbotix_descriptions/urdf/wx250s.urdf.xacro (robot description, xacro)
@@ -131,5 +131,5 @@
   <link name="$(arg robot_name)/upper_forearm_link">
     <visual>
-      <origin rpy="0 0 ${-pi/2}" xyz="0.24766 0 0"/>
+      <origin rpy="0 0 0" xyz="0 0 0"/>
       <geometry>
         <mesh filename="package://interbotix_descriptions/meshes/meshes_wx250s/WXSA-250-M-4-UF.stl" scale="0.001 0.001 0.001"/>
@@ -138,5 +138,5 @@
     </visual>
     <collision>
-      <origin rpy="0 0 ${-pi/2}" xyz="0.24766 0 0"/>
+      <origin rpy="0 0 0" xyz="0 0 0"/>
       <geometry>
         <mesh filename="package://interbotix_descriptions/meshes/meshes_wx250s/WXSA-250-M-4-UF.stl" scale="0.001 0.001 0.001"/>
@@ -144,7 +144,7 @@
     </collision>
     <inertial>
-      <origin rpy="0 0 ${-pi/2}" xyz="0 0 0"/>
-      <mass value="0.1" />
-      <inertia ixx="0.005" iyy="0.0002" izz="0.005" ixy="0" ixz="0" iyz="0" />
+      <origin rpy="0 0 0" xyz="0.1079630000 0.0001158760 0"/>
+      <mass value="0.234589" />
+      <inertia ixx="0.0000397100" iyy="0.0008878000" izz="0.0008880000" ixy="0.0000023528" ixz="0" iyz="0" />
     </inertial>
   </link>
@@ -152,5 +152,5 @@
     <axis xyz="1 0 0"/>
     <limit effort="100" lower="${radians(-180)}" upper="${radians(180)}" velocity="${pi}"/>
-    <origin rpy="0 0 0" xyz="0.1721 0 0"/>
+    <origin rpy="0 0 0" xyz="0.175 0 0"/>
     <parent link="$(arg robot_name)/upper_forearm_link"/>
     <child link="$(arg robot_name)/lower_forearm_link"/>
@@ -167,5 +167,5 @@
   <link name="$(arg robot_name)/lower_forearm_link">
     <visual>
-      <origin rpy="0 ${-pi/2} ${-pi/2}" xyz="0.07545 0 0"/>
+      <origin rpy="0 0 0" xyz="0 0 0"/>
       <geometry>
         <mesh filename="package://interbotix_descriptions/meshes/meshes_wx250s/WXSA-250-M-5-LF.stl" scale="0.001 0.001 0.001"/>
@@ -174,5 +174,5 @@
     </visual>
     <collision>
-      <origin rpy="0 ${-pi/2} ${-pi/2}" xyz="0.07545 0 0"/>
+      <origin rpy="0 0 0" xyz="0 0 0"/>
       <geometry>
         <mesh filename="package://interbotix_descriptions/meshes/meshes_wx250s/WXSA-250-M-5-LF.stl" scale="0.001 0.001 0.001"/>
@@ -180,7 +180,7 @@
     </collision>
     <inertial>
-      <origin rpy="0 ${-pi/2} ${-pi/2}" xyz="0 0 0"/>
-      <mass value="0.1" />
-      <inertia ixx="0.005" iyy="0.0002" izz="0.005" ixy="0" ixz="0" iyz="0" />
+      <origin rpy="0 0 0" xyz="0.0374395000 -0.0052225200 0"/>
+      <mass value="0.220991" />
+      <inertia ixx="0.0000636900" iyy="0.0001677000" izz="0.0001834000" ixy="-0.0000229200" ixz="0" iyz="0" />
     </inertial>
   </link>
@@ -188,5 +188,5 @@
     <axis xyz="0 1 0"/>
     <limit effort="100" lower="${radians(-123)}" upper="${radians(100)}" velocity="${pi}"/>
-    <origin rpy="0 0 0" xyz="0.07779 0 0"/>
+    <origin rpy="0 0 0" xyz="0.075 0 0"/>
     <parent link="$(arg robot_name)/lower_forearm_link"/>
     <child link="$(arg robot_name)/wrist_link"/>
