Commit message: Updated all ROS packages to be equivalent to the ones in the interbotix_ros_arms repo. Also added python_demos directory if a user would like to control a platform without a controller and does not want to make their own custom ROS package

File: interbotix_descriptions/urdf/px100.urdf.xacro (robot description, xacro)
@@ -2,11 +2,11 @@
 <robot name="px100" xmlns:xacro="http://ros.org/wiki/xacro">
   <xacro:arg name="robot_name" default = ""/>
-  <xacro:arg name="default_gripper_bar" default="true"/>
-  <xacro:arg name="default_gripper_fingers" default="true"/>
-  <xacro:arg name="external_gripper_urdf" default="false"/>
-  <xacro:arg name="external_gripper_urdf_loc" default=""/>
-  <xacro:arg name="gazebo" default="false"/>
-  <xacro:arg name="moveit" default="false"/>
-  <xacro:if value="$(arg gazebo)">
+  <xacro:arg name="use_world_frame" default="false"/>
+  <xacro:arg name="use_default_gripper_bar" default="true"/>
+  <xacro:arg name="use_default_gripper_fingers" default="true"/>
+  <xacro:arg name="external_urdf_loc" default=""/>
+  <xacro:arg name="load_gazebo_configs" default="false"/>
+  <xacro:property name="urdf_loc" value="$(arg external_urdf_loc)"/>
+  <xacro:if value="$(arg load_gazebo_configs)">
     <xacro:include filename="$(find interbotix_gazebo)/config/interbotix_texture.gazebo"/>
   </xacro:if>
@@ -14,5 +14,5 @@
     <texture filename="package://interbotix_descriptions/meshes/interbotix_black.png"/>
   </material>
-  <xacro:if value="$(arg moveit)">
+  <xacro:if value="$(arg use_world_frame)">
     <link name="world"/>
     <joint name="fixed" type="fixed">
@@ -234,5 +234,5 @@
   </link>
   <!-- If the default gripper bar is being used, then also add the gripper bar -->
-  <xacro:if value="$(arg default_gripper_bar)">
+  <xacro:if value="$(arg use_default_gripper_bar)">
     <joint name="gripper_bar" type="fixed">
       <axis xyz="1 0 0"/>
@@ -274,5 +274,5 @@
     </link>
     <!-- If the default gripper fingers are being used, add those as well -->
-    <xacro:if value="$(arg default_gripper_fingers)">
+    <xacro:if value="$(arg use_default_gripper_fingers)">
       <joint name="left_finger" type="prismatic">
         <axis xyz="0 1 0"/>
@@ -317,5 +317,5 @@
         <parent link="$(arg robot_name)/fingers_link"/>
         <child link="$(arg robot_name)/right_finger_link"/>
-        <xacro:unless value="$(arg gazebo)">
+        <xacro:unless value="$(arg load_gazebo_configs)">
           <mimic joint="left_finger" multiplier="-1" offset="0"/>
         </xacro:unless>
@@ -364,6 +364,6 @@
     </xacro:if>
   </xacro:if>
-  <xacro:if value="$(arg external_gripper_urdf)">
-    <xacro:include filename="$(arg external_gripper_urdf_loc)"/>
+  <xacro:if value="${urdf_loc != ''}">
+    <xacro:include filename="${urdf_loc}"/>
   </xacro:if>
 </robot>

File: interbotix_descriptions/urdf/px150.urdf.xacro (robot description, xacro)
@@ -2,11 +2,11 @@
 <robot name="px150" xmlns:xacro="http://ros.org/wiki/xacro">
   <xacro:arg name="robot_name" default = ""/>
-  <xacro:arg name="default_gripper_bar" default="true"/>
-  <xacro:arg name="default_gripper_fingers" default="true"/>
-  <xacro:arg name="external_gripper_urdf" default="false"/>
-  <xacro:arg name="external_gripper_urdf_loc" default=""/>
-  <xacro:arg name="gazebo" default="false"/>
-  <xacro:arg name="moveit" default="false"/>
-  <xacro:if value="$(arg gazebo)">
+  <xacro:arg name="use_world_frame" default="false"/>
+  <xacro:arg name="use_default_gripper_bar" default="true"/>
+  <xacro:arg name="use_default_gripper_fingers" default="true"/>
+  <xacro:arg name="external_urdf_loc" default=""/>
+  <xacro:arg name="load_gazebo_configs" default="false"/>
+  <xacro:property name="urdf_loc" value="$(arg external_urdf_loc)"/>
+  <xacro:if value="$(arg load_gazebo_configs)">
     <xacro:include filename="$(find interbotix_gazebo)/config/interbotix_texture.gazebo"/>
   </xacro:if>
@@ -14,5 +14,5 @@
     <texture filename="package://interbotix_descriptions/meshes/interbotix_black.png"/>
   </material>
-  <xacro:if value="$(arg moveit)">
+  <xacro:if value="$(arg use_world_frame)">
     <link name="world"/>
     <joint name="fixed" type="fixed">
@@ -270,5 +270,5 @@
   </link>
   <!-- If the default gripper bar is being used, then also add the gripper bar -->
-  <xacro:if value="$(arg default_gripper_bar)">
+  <xacro:if value="$(arg use_default_gripper_bar)">
     <joint name="gripper_bar" type="fixed">
       <axis xyz="1 0 0"/>
@@ -310,5 +310,5 @@
     </link>
     <!-- If the default gripper fingers are being used, add those as well -->
-    <xacro:if value="$(arg default_gripper_fingers)">
+    <xacro:if value="$(arg use_default_gripper_fingers)">
       <joint name="left_finger" type="prismatic">
         <axis xyz="0 1 0"/>
@@ -353,5 +353,5 @@
         <parent link="$(arg robot_name)/fingers_link"/>
         <child link="$(arg robot_name)/right_finger_link"/>
-        <xacro:unless value="$(arg gazebo)">
+        <xacro:unless value="$(arg load_gazebo_configs)">
           <mimic joint="left_finger" multiplier="-1" offset="0"/>
         </xacro:unless>
@@ -400,6 +400,6 @@
     </xacro:if>
   </xacro:if>
-  <xacro:if value="$(arg external_gripper_urdf)">
-    <xacro:include filename="$(arg external_gripper_urdf_loc)"/>
+  <xacro:if value="${urdf_loc != ''}">
+    <xacro:include filename="${urdf_loc}"/>
   </xacro:if>
 </robot>

File: interbotix_descriptions/urdf/pxxls.urdf.xacro (robot description, xacro)
@@ -2,9 +2,17 @@
 <robot name="pxxls" xmlns:xacro="http://ros.org/wiki/xacro">
   <xacro:arg name="robot_name" default = ""/>
-  <xacro:arg name="external_gripper_urdf" default="false"/>
-  <xacro:arg name="external_gripper_urdf_loc" default=""/>
+  <xacro:arg name="external_urdf_loc" default=""/>
+  <xacro:arg name="use_world_frame" default="false"/>
+  <xacro:property name="urdf_loc" value="$(arg external_urdf_loc)"/>
   <material name="interbotix_black">
     <texture filename="package://interbotix_descriptions/meshes/interbotix_black.png"/>
   </material>
+  <xacro:if value="$(arg use_world_frame)">
+    <link name="world"/>
+    <joint name="fixed" type="fixed">
+      <parent link="world"/>
+      <child link="$(arg robot_name)/base_link"/>
+    </joint>
+  </xacro:if>
   <link name="$(arg robot_name)/base_link">
     <visual>
@@ -74,6 +82,6 @@
   <link name="$(arg robot_name)/surface_link">
   </link>
-  <xacro:if value="$(arg external_gripper_urdf)">
-    <xacro:include filename="$(arg external_gripper_urdf_loc)"/>
+  <xacro:if value="${urdf_loc != ''}">
+    <xacro:include filename="${urdf_loc}"/>
   </xacro:if>
 </robot>

File: interbotix_descriptions/urdf/rx150.urdf.xacro (robot description, xacro)
@@ -2,11 +2,11 @@
 <robot name="rx150" xmlns:xacro="http://ros.org/wiki/xacro">
   <xacro:arg name="robot_name" default = ""/>
-  <xacro:arg name="default_gripper_bar" default="true"/>
-  <xacro:arg name="default_gripper_fingers" default="true"/>
-  <xacro:arg name="external_gripper_urdf" default="false"/>
-  <xacro:arg name="external_gripper_urdf_loc" default=""/>
-  <xacro:arg name="gazebo" default="false"/>
-  <xacro:arg name="moveit" default="false"/>
-  <xacro:if value="$(arg gazebo)">
+  <xacro:arg name="use_world_frame" default="false"/>
+  <xacro:arg name="use_default_gripper_bar" default="true"/>
+  <xacro:arg name="use_default_gripper_fingers" default="true"/>
+  <xacro:arg name="external_urdf_loc" default=""/>
+  <xacro:arg name="load_gazebo_configs" default="false"/>
+  <xacro:property name="urdf_loc" value="$(arg external_urdf_loc)"/>
+  <xacro:if value="$(arg load_gazebo_configs)">
     <xacro:include filename="$(find interbotix_gazebo)/config/interbotix_texture.gazebo"/>
   </xacro:if>
@@ -14,5 +14,5 @@
     <texture filename="package://interbotix_descriptions/meshes/interbotix_black.png"/>
   </material>
-  <xacro:if value="$(arg moveit)">
+  <xacro:if value="$(arg use_world_frame)">
     <link name="world"/>
     <joint name="fixed" type="fixed">
@@ -270,5 +270,5 @@
   </link>
   <!-- If the default gripper bar is being used, then also add the gripper bar -->
-  <xacro:if value="$(arg default_gripper_bar)">
+  <xacro:if value="$(arg use_default_gripper_bar)">
     <joint name="gripper_bar" type="fixed">
       <axis xyz="1 0 0"/>
@@ -310,5 +310,5 @@
     </link>
     <!-- If the default gripper fingers are being used, add those as well -->
-    <xacro:if value="$(arg default_gripper_fingers)">
+    <xacro:if value="$(arg use_default_gripper_fingers)">
       <joint name="left_finger" type="prismatic">
         <axis xyz="0 1 0"/>
@@ -353,5 +353,5 @@
         <parent link="$(arg robot_name)/fingers_link"/>
         <child link="$(arg robot_name)/right_finger_link"/>
-        <xacro:unless value="$(arg gazebo)">
+        <xacro:unless value="$(arg load_gazebo_configs)">
           <mimic joint="left_finger" multiplier="-1" offset="0"/>
         </xacro:unless>
@@ -400,6 +400,6 @@
     </xacro:if>
   </xacro:if>
-  <xacro:if value="$(arg external_gripper_urdf)">
-    <xacro:include filename="$(arg external_gripper_urdf_loc)"/>
+  <xacro:if value="${urdf_loc != ''}">
+    <xacro:include filename="${urdf_loc}"/>
   </xacro:if>
 </robot>

File: interbotix_descriptions/urdf/rx200.urdf.xacro (robot description, xacro)
@@ -2,11 +2,11 @@
 <robot name="rx200" xmlns:xacro="http://ros.org/wiki/xacro">
   <xacro:arg name="robot_name" default = ""/>
-  <xacro:arg name="default_gripper_bar" default="true"/>
-  <xacro:arg name="default_gripper_fingers" default="true"/>
-  <xacro:arg name="external_gripper_urdf" default="false"/>
-  <xacro:arg name="external_gripper_urdf_loc" default=""/>
-  <xacro:arg name="gazebo" default="false"/>
-  <xacro:arg name="moveit" default="false"/>
-  <xacro:if value="$(arg gazebo)">
+  <xacro:arg name="use_world_frame" default="false"/>
+  <xacro:arg name="use_default_gripper_bar" default="true"/>
+  <xacro:arg name="use_default_gripper_fingers" default="true"/>
+  <xacro:arg name="external_urdf_loc" default=""/>
+  <xacro:arg name="load_gazebo_configs" default="false"/>
+  <xacro:property name="urdf_loc" value="$(arg external_urdf_loc)"/>
+  <xacro:if value="$(arg load_gazebo_configs)">
     <xacro:include filename="$(find interbotix_gazebo)/config/interbotix_texture.gazebo"/>
   </xacro:if>
@@ -14,5 +14,5 @@
     <texture filename="package://interbotix_descriptions/meshes/interbotix_black.png"/>
   </material>
-  <xacro:if value="$(arg moveit)">
+  <xacro:if value="$(arg use_world_frame)">
     <link name="world"/>
     <joint name="fixed" type="fixed">
@@ -270,5 +270,5 @@
   </link>
   <!-- If the default gripper bar is being used, then also add the gripper bar -->
-  <xacro:if value="$(arg default_gripper_bar)">
+  <xacro:if value="$(arg use_default_gripper_bar)">
     <joint name="gripper_bar" type="fixed">
       <axis xyz="1 0 0"/>
@@ -310,5 +310,5 @@
     </link>
     <!-- If the default gripper fingers are being used, add those as well -->
-    <xacro:if value="$(arg default_gripper_fingers)">
+    <xacro:if value="$(arg use_default_gripper_fingers)">
       <joint name="left_finger" type="prismatic">
         <axis xyz="0 1 0"/>
@@ -353,5 +353,5 @@
         <parent link="$(arg robot_name)/fingers_link"/>
         <child link="$(arg robot_name)/right_finger_link"/>
-        <xacro:unless value="$(arg gazebo)">
+        <xacro:unless value="$(arg load_gazebo_configs)">
           <mimic joint="left_finger" multiplier="-1" offset="0"/>
         </xacro:unless>
@@ -400,6 +400,6 @@
     </xacro:if>
   </xacro:if>
-  <xacro:if value="$(arg external_gripper_urdf)">
-    <xacro:include filename="$(arg external_gripper_urdf_loc)"/>
+  <xacro:if value="${urdf_loc != ''}">
+    <xacro:include filename="${urdf_loc}"/>
   </xacro:if>
 </robot>

File: interbotix_descriptions/urdf/vx250.urdf.xacro (robot description, xacro)
@@ -2,11 +2,11 @@
 <robot name="vx250" xmlns:xacro="http://ros.org/wiki/xacro">
   <xacro:arg name="robot_name" default = ""/>
-  <xacro:arg name="default_gripper_bar" default="true"/>
-  <xacro:arg name="default_gripper_fingers" default="true"/>
-  <xacro:arg name="external_gripper_urdf" default="false"/>
-  <xacro:arg name="external_gripper_urdf_loc" default=""/>
-  <xacro:arg name="gazebo" default="false"/>
-  <xacro:arg name="moveit" default="false"/>
-  <xacro:if value="$(arg gazebo)">
+  <xacro:arg name="use_world_frame" default="false"/>
+  <xacro:arg name="use_default_gripper_bar" default="true"/>
+  <xacro:arg name="use_default_gripper_fingers" default="true"/>
+  <xacro:arg name="external_urdf_loc" default=""/>
+  <xacro:arg name="load_gazebo_configs" default="false"/>
+  <xacro:property name="urdf_loc" value="$(arg external_urdf_loc)"/>
+  <xacro:if value="$(arg load_gazebo_configs)">
     <xacro:include filename="$(find interbotix_gazebo)/config/interbotix_texture.gazebo"/>
   </xacro:if>
@@ -14,5 +14,5 @@
     <texture filename="package://interbotix_descriptions/meshes/interbotix_black.png"/>
   </material>
-  <xacro:if value="$(arg moveit)">
+  <xacro:if value="$(arg use_world_frame)">
     <link name="world"/>
     <joint name="fixed" type="fixed">
@@ -270,5 +270,5 @@
   </link>
   <!-- If the default gripper bar is being used, then also add the gripper bar -->
-  <xacro:if value="$(arg default_gripper_bar)">
+  <xacro:if value="$(arg use_default_gripper_bar)">
     <joint name="gripper_bar" type="fixed">
       <axis xyz="1 0 0"/>
@@ -310,5 +310,5 @@
     </link>
     <!-- If the default gripper fingers are being used, add those as well -->
-    <xacro:if value="$(arg default_gripper_fingers)">
+    <xacro:if value="$(arg use_default_gripper_fingers)">
       <joint name="left_finger" type="prismatic">
         <axis xyz="0 1 0"/>
@@ -353,5 +353,5 @@
         <parent link="$(arg robot_name)/fingers_link"/>
         <child link="$(arg robot_name)/right_finger_link"/>
-        <xacro:unless value="$(arg gazebo)">
+        <xacro:unless value="$(arg load_gazebo_configs)">
           <mimic joint="left_finger" multiplier="-1" offset="0"/>
         </xacro:unless>
@@ -400,6 +400,6 @@
     </xacro:if>
   </xacro:if>
-  <xacro:if value="$(arg external_gripper_urdf)">
-    <xacro:include filename="$(arg external_gripper_urdf_loc)"/>
+  <xacro:if value="${urdf_loc != ''}">
+    <xacro:include filename="${urdf_loc}"/>
   </xacro:if>
 </robot>

File: interbotix_descriptions/urdf/vx300.urdf.xacro (robot description, xacro)
@@ -2,11 +2,11 @@
 <robot name="vx300" xmlns:xacro="http://ros.org/wiki/xacro">
   <xacro:arg name="robot_name" default = ""/>
-  <xacro:arg name="default_gripper_bar" default="true"/>
-  <xacro:arg name="default_gripper_fingers" default="true"/>
-  <xacro:arg name="external_gripper_urdf" default="false"/>
-  <xacro:arg name="external_gripper_urdf_loc" default=""/>
-  <xacro:arg name="gazebo" default="false"/>
-  <xacro:arg name="moveit" default="false"/>
-  <xacro:if value="$(arg gazebo)">
+  <xacro:arg name="use_world_frame" default="false"/>
+  <xacro:arg name="use_default_gripper_bar" default="true"/>
+  <xacro:arg name="use_default_gripper_fingers" default="true"/>
+  <xacro:arg name="external_urdf_loc" default=""/>
+  <xacro:arg name="load_gazebo_configs" default="false"/>
+  <xacro:property name="urdf_loc" value="$(arg external_urdf_loc)"/>
+  <xacro:if value="$(arg load_gazebo_configs)">
     <xacro:include filename="$(find interbotix_gazebo)/config/interbotix_texture.gazebo"/>
   </xacro:if>
@@ -14,5 +14,5 @@
     <texture filename="package://interbotix_descriptions/meshes/interbotix_black.png"/>
   </material>
-  <xacro:if value="$(arg moveit)">
+  <xacro:if value="$(arg use_world_frame)">
     <link name="world"/>
     <joint name="fixed" type="fixed">
@@ -270,5 +270,5 @@
   </link>
   <!-- If the default gripper bar is being used, then also add the gripper bar -->
-  <xacro:if value="$(arg default_gripper_bar)">
+  <xacro:if value="$(arg use_default_gripper_bar)">
     <joint name="gripper_bar" type="fixed">
       <axis xyz="1 0 0"/>
@@ -310,5 +310,5 @@
     </link>
     <!-- If the default gripper fingers are being used, add those as well -->
-    <xacro:if value="$(arg default_gripper_fingers)">
+    <xacro:if value="$(arg use_default_gripper_fingers)">
       <joint name="left_finger" type="prismatic">
         <axis xyz="0 1 0"/>
@@ -353,5 +353,5 @@
         <parent link="$(arg robot_name)/fingers_link"/>
         <child link="$(arg robot_name)/right_finger_link"/>
-        <xacro:unless value="$(arg gazebo)">
+        <xacro:unless value="$(arg load_gazebo_configs)">
           <mimic joint="left_finger" multiplier="-1" offset="0"/>
         </xacro:unless>
@@ -400,6 +400,6 @@
     </xacro:if>
   </xacro:if>
-  <xacro:if value="$(arg external_gripper_urdf)">
-    <xacro:include filename="$(arg external_gripper_urdf_loc)"/>
+  <xacro:if value="${urdf_loc != ''}">
+    <xacro:include filename="${urdf_loc}"/>
   </xacro:if>
 </robot>

File: interbotix_descriptions/urdf/vx300s.urdf.xacro (robot description, xacro)
@@ -2,11 +2,11 @@
 <robot name="vx300s" xmlns:xacro="http://ros.org/wiki/xacro">
   <xacro:arg name="robot_name" default = ""/>
-  <xacro:arg name="default_gripper_bar" default="true"/>
-  <xacro:arg name="default_gripper_fingers" default="true"/>
-  <xacro:arg name="external_gripper_urdf" default="false"/>
-  <xacro:arg name="external_gripper_urdf_loc" default=""/>
-  <xacro:arg name="gazebo" default="false"/>
-  <xacro:arg name="moveit" default="false"/>
-  <xacro:if value="$(arg gazebo)">
+  <xacro:arg name="use_world_frame" default="false"/>
+  <xacro:arg name="use_default_gripper_bar" default="true"/>
+  <xacro:arg name="use_default_gripper_fingers" default="true"/>
+  <xacro:arg name="external_urdf_loc" default=""/>
+  <xacro:arg name="load_gazebo_configs" default="false"/>
+  <xacro:property name="urdf_loc" value="$(arg external_urdf_loc)"/>
+  <xacro:if value="$(arg load_gazebo_configs)">
     <xacro:include filename="$(find interbotix_gazebo)/config/interbotix_texture.gazebo"/>
   </xacro:if>
@@ -14,5 +14,5 @@
     <texture filename="package://interbotix_descriptions/meshes/interbotix_black.png"/>
   </material>
-  <xacro:if value="$(arg moveit)">
+  <xacro:if value="$(arg use_world_frame)">
     <link name="world"/>
     <joint name="fixed" type="fixed">
@@ -306,5 +306,5 @@
   </link>
   <!-- If the default gripper bar is being used, then also add the gripper bar -->
-  <xacro:if value="$(arg default_gripper_bar)">
+  <xacro:if value="$(arg use_default_gripper_bar)">
     <joint name="gripper_bar" type="fixed">
       <axis xyz="1 0 0"/>
@@ -346,5 +346,5 @@
     </link>
     <!-- If the default gripper fingers are being used, add those as well -->
-    <xacro:if value="$(arg default_gripper_fingers)">
+    <xacro:if value="$(arg use_default_gripper_fingers)">
       <joint name="left_finger" type="prismatic">
         <axis xyz="0 1 0"/>
@@ -389,5 +389,5 @@
         <parent link="$(arg robot_name)/fingers_link"/>
         <child link="$(arg robot_name)/right_finger_link"/>
-        <xacro:unless value="$(arg gazebo)">
+        <xacro:unless value="$(arg load_gazebo_configs)">
           <mimic joint="left_finger" multiplier="-1" offset="0"/>
         </xacro:unless>
@@ -436,6 +436,6 @@
     </xacro:if>
   </xacro:if>
-  <xacro:if value="$(arg external_gripper_urdf)">
-    <xacro:include filename="$(arg external_gripper_urdf_loc)"/>
+  <xacro:if value="${urdf_loc != ''}">
+    <xacro:include filename="${urdf_loc}"/>
   </xacro:if>
 </robot>

File: interbotix_descriptions/urdf/vxxmd.urdf.xacro (robot description, xacro)
@@ -2,9 +2,17 @@
 <robot name="vxxmd" xmlns:xacro="http://ros.org/wiki/xacro">
   <xacro:arg name="robot_name" default = ""/>
-  <xacro:arg name="external_gripper_urdf" default="false"/>
-  <xacro:arg name="external_gripper_urdf_loc" default=""/>
+  <xacro:arg name="external_urdf_loc" default=""/>
+  <xacro:arg name="use_world_frame" default="false"/>
+  <xacro:property name="urdf_loc" value="$(arg external_urdf_loc)"/>
   <material name="interbotix_black">
     <texture filename="package://interbotix_descriptions/meshes/interbotix_black.png"/>
   </material>
+  <xacro:if value="$(arg use_world_frame)">
+    <link name="world"/>
+    <joint name="fixed" type="fixed">
+      <parent link="world"/>
+      <child link="$(arg robot_name)/base_link"/>
+    </joint>
+  </xacro:if>
   <link name="$(arg robot_name)/base_link">
     <visual>
@@ -74,6 +82,6 @@
   <link name="$(arg robot_name)/surface_link">
   </link>
-  <xacro:if value="$(arg external_gripper_urdf)">
-    <xacro:include filename="$(arg external_gripper_urdf_loc)"/>
+  <xacro:if value="${urdf_loc != ''}">
+    <xacro:include filename="${urdf_loc}"/>
   </xacro:if>
 </robot>

File: interbotix_descriptions/urdf/vxxms.urdf.xacro (robot description, xacro)
@@ -2,9 +2,17 @@
 <robot name="vxxms" xmlns:xacro="http://ros.org/wiki/xacro">
   <xacro:arg name="robot_name" default = ""/>
-  <xacro:arg name="external_gripper_urdf" default="false"/>
-  <xacro:arg name="external_gripper_urdf_loc" default=""/>
+  <xacro:arg name="external_urdf_loc" default=""/>
+  <xacro:arg name="use_world_frame" default="false"/>
+  <xacro:property name="urdf_loc" value="$(arg external_urdf_loc)"/>
   <material name="interbotix_black">
     <texture filename="package://interbotix_descriptions/meshes/interbotix_black.png"/>
   </material>
+  <xacro:if value="$(arg use_world_frame)">
+    <link name="world"/>
+    <joint name="fixed" type="fixed">
+      <parent link="world"/>
+      <child link="$(arg robot_name)/base_link"/>
+    </joint>
+  </xacro:if>
   <link name="$(arg robot_name)/base_link">
     <visual>
@@ -74,6 +82,6 @@
   <link name="$(arg robot_name)/surface_link">
   </link>
-  <xacro:if value="$(arg external_gripper_urdf)">
-    <xacro:include filename="$(arg external_gripper_urdf_loc)"/>
+  <xacro:if value="${urdf_loc != ''}">
+    <xacro:include filename="${urdf_loc}"/>
   </xacro:if>
 </robot>
